File: Power Supply.kicad_pcb (KiCad board)
At the start: 2 copper layers, 75 x 70 mm, 16 parts

Commit message: re-routing
Routing:
- net Net-(220v_AC1-Pin_1): track 53.6 -> 54.5 mm
Changed lines of the file:
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@@
 	)
 	(segment
-		(start 65 79.5)
-		(end 65.5 80)
+		(start 64.5 114)
+		(end 71 120.5)
 		(width 2)
 		(layer "F.Cu")
@@
 	)
 	(segment
-		(start 67.55 76.95)
-		(end 65 79.5)
+		(start 64.5 79.5)
+		(end 64.5 114)
 		(width 2)
 		(layer "F.Cu")
@@
 	)
 	(segment
-		(start 74.92 113.92)
+		(start 71 120.5)
 		(end 74.92 120.5)
 		(width 2)
@@
 	)
 	(segment
-		(start 71.5 110.5)
-		(end 74.92 113.92)
+		(start 70.37 76.95)
+		(end 67.05 76.95)
 		(width 2)
 		(layer "F.Cu")
@@
 	)
 	(segment
-		(start 65.5 108)
-		(end 68 110.5)
+		(start 67.05 76.95)
+		(end 64.5 79.5)
 		(width 2)
 		(layer "F.Cu")
-		(net 4)
-	)
-	(segment
-		(start 68 110.5)
-		(end 71.5 110.5)
-		(width 2)
-		(layer "F.Cu")
-		(net 4)
-	)
-	(segment
-		(start 70.37 76.95)
-		(end 67.55 76.95)
-		(width 2)
-		(layer "F.Cu")
-		(net 4)
-	)
-	(segment
-		(start 65.5 80)
-		(end 65.5 108)
-		(width 2)
-		(layer "F.Cu")
