File: Power Supply.kicad_pcb (KiCad board)
At the start: 2 copper layers, 75 x 70 mm, 16 parts

Commit message: Added Copper fill in back-layer
Connections:
- net Net-(12v_DC1-Pin_1) renamed GND
Routing:
- added copper zone on B.Cu, net GND
Changed lines of the file:
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@@
 	(net 0 "")
 	(net 1 "Net-(12v_DC1-Pin_2)")
-	(net 2 "Net-(12v_DC1-Pin_1)")
+	(net 2 "GND")
 	(net 3 "Net-(220v_AC1-Pin_2)")
 	(net 4 "Net-(220v_AC1-Pin_1)")
@@
 			(layers "*.Cu" "*.Mask")
 			(remove_unused_layers no)
-			(net 2 "Net-(12v_DC1-Pin_1)")
+			(net 2 "GND")
 			(pintype "passive")
 		)
@@
 			(remove_unused_layers no)
 			(roundrect_rratio 0.120192)
-			(net 2 "Net-(12v_DC1-Pin_1)")
+			(net 2 "GND")
 			(pinfunction "Pin_1")
 			(pintype "passive")
@@
 			(layers "*.Cu" "*.Mask")
 			(remove_unused_layers no)
-			(net 2 "Net-(12v_DC1-Pin_1)")
+			(net 2 "GND")
 			(pinfunction "A")
 			(pintype "passive")
@@
 			(layers "*.Cu" "*.Mask")
 			(remove_unused_layers no)
-			(net 2 "Net-(12v_DC1-Pin_1)")
+			(net 2 "GND")
 			(pintype "passive")
 		)
@@
 			(layers "*.Cu" "*.Mask")
 			(remove_unused_layers no)
-			(net 2 "Net-(12v_DC1-Pin_1)")
+			(net 2 "GND")
 			(pinfunction "A")
 			(pintype "passive")
@@
 		(net 10)
 	)
+	(zone
+		(net 2)
+		(net_name "GND")
+		(layer "B.Cu")
+		(hatch edge 0.5)
+		(connect_pads
+			(clearance 0.5)
+		)
+		(min_thickness 0.25)
+		(filled_areas_thickness no)
+		(fill yes
+			(thermal_gap 0.5)
+			(thermal_bridge_width 0.5)
+		)
+		(polygon
+			(pts
+				(xy 57.5 59.5) (xy 136 59.5) (xy 136 130.5) (xy 58 130.5) (xy 57.5 130)
+			)
+		)
+	)
 	(embedded_fonts no)
